File: wireless-power-transfer/primary/KiCad/tank.sch (KiCad schematic (older format))
At the start: 9 parts

Commit message: Schematics and footprint libraries ready
Parts:
- Cf1, Cf2, Cr1, Cr2: footprint (none) -> footprint:C_Rect_L18.0mm_W5.0mm_P15.00mm_FKS3_FKP3
- Jf1, Jin1, Jr1, Jr2: footprint (none) -> footprint:TerminalBlock_Pheonix_MKDS1.5-2pol
- Lf1: footprint componentesGIT:MuRata 1500 47u -> footprint:MuRata 1500 47u
Connections:
- net at Cf1.2, Jf1.2, Lf1.2: now also Cf2.1; no longer Cf2.2
- net at Cf1.1, Cr1.2, Cr2.2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: now also Cf2.2; no longer Cf2.1
Changed lines of the file:
@@
 Comment4 ""
 $EndDescr
-$Comp
-L L Lf1
-U 1 1 59F1AF47
-P 3500 4150
-F 0 "Lf1" V 3450 4150 50  0000 C CNN
-F 1 "47uH" V 3575 4150 50  0000 C CNN
-F 2 "componentesGIT:MuRata 1500 47u" H 3500 4150 50  0001 C CNN
-F 3 "" H 3500 4150 50  0001 C CNN
-	1    3500 4150
-	0    -1   -1   0
-$EndComp
 Wire Wire Line
 	3000 4400 3000 4150
@@
 F 0 "Jin1" H 2800 4750 50  0000 C TNN
 F 1 "Screw_Terminal_1x02" V 2650 4500 50  0000 C TNN
-F 2 "" H 2800 4275 50  0001 C CNN
+F 2 "footprint:TerminalBlock_Pheonix_MKDS1.5-2pol" H 2800 4275 50  0001 C CNN
 F 3 "" H 2775 4500 50  0001 C CNN
 	1    2800 4500
@@
 F 0 "Jf1" H 3500 3950 50  0000 C TNN
 F 1 "Screw_Terminal_1x02" V 3350 3700 50  0000 C TNN
-F 2 "" H 3500 3475 50  0001 C CNN
+F 2 "footprint:TerminalBlock_Pheonix_MKDS1.5-2pol" H 3500 3475 50  0001 C CNN
 F 3 "" H 3475 3700 50  0001 C CNN
 	1    3500 3700
@@
 F 0 "Cf1" H 4175 4250 50  0000 L CNN
 F 1 "C" H 4175 4050 50  0000 L CNN
-F 2 "" H 4188 4000 50  0001 C CNN
+F 2 "footprint:C_Rect_L18.0mm_W5.0mm_P15.00mm_FKS3_FKP3" H 4188 4000 50  0001 C CNN
 F 3 "" H 4150 4150 50  0001 C CNN
 	1    4150 4150
@@
 F 0 "Cf2" H 4175 4600 50  0000 L CNN
 F 1 "C" H 4175 4400 50  0000 L CNN
-F 2 "" H 4188 4350 50  0001 C CNN
+F 2 "footprint:C_Rect_L18.0mm_W5.0mm_P15.00mm_FKS3_FKP3" H 4188 4350 50  0001 C CNN
 F 3 "" H 4150 4500 50  0001 C CNN
 	1    4150 4500
-	0    1    1    0
+	0    -1   -1   0
 $EndComp
 $Comp
@@
 F 0 "Cr1" H 4775 4550 50  0000 L CNN
 F 1 "C" H 4775 4350 50  0000 L CNN
-F 2 "" H 4788 4300 50  0001 C CNN
+F 2 "footprint:C_Rect_L18.0mm_W5.0mm_P15.00mm_FKS3_FKP3" H 4788 4300 50  0001 C CNN
 F 3 "" H 4750 4450 50  0001 C CNN
 	1    4750 4450
@@
 F 0 "Cr2" H 5125 4550 50  0000 L CNN
 F 1 "C" H 5125 4350 50  0000 L CNN
-F 2 "" H 5138 4300 50  0001 C CNN
+F 2 "footprint:C_Rect_L18.0mm_W5.0mm_P15.00mm_FKS3_FKP3" H 5138 4300 50  0001 C CNN
 F 3 "" H 5100 4450 50  0001 C CNN
 	1    5100 4450
@@
 F 0 "Jr1" H 5950 4400 50  0000 C TNN
 F 1 "Screw_Terminal_1x02" V 5800 4150 50  0000 C TNN
-F 2 "" H 5950 3925 50  0001 C CNN
+F 2 "footprint:TerminalBlock_Pheonix_MKDS1.5-2pol" H 5950 3925 50  0001 C CNN
 F 3 "" H 5925 4150 50  0001 C CNN
 	1    5950 4150
@@
 F 0 "Jr2" H 5975 5000 50  0000 C TNN
 F 1 "Screw_Terminal_1x02" V 5825 4750 50  0000 C TNN
-F 2 "" H 5975 4525 50  0001 C CNN
+F 2 "footprint:TerminalBlock_Pheonix_MKDS1.5-2pol" H 5975 4525 50  0001 C CNN
 F 3 "" H 5950 4750 50  0001 C CNN
 	1    5975 4750
 	-1   0    0    -1
 $EndComp
+$Comp
+L L Lf1
+U 1 1 5AA74506
+P 3500 4150
+F 0 "Lf1" V 3450 4150 50  0000 C CNN
+F 1 "47uH" V 3575 4150 50  0000 C CNN
+F 2 "footprint:MuRata 1500 47u" H 3500 4150 50  0001 C CNN
+F 3 "" H 3500 4150 50  0001 C CNN
+	1    3500 4150
+	0    -1   -1   0
+$EndComp
 $EndSCHEMATC
