File: wireless-power-transfer/primary/KiCad/tfg.kicad_pcb (KiCad board)
At the start: 2 copper layers, 160 x 100 mm, 57 parts, among them J1 CONN_01X06, J2 Screw_Terminal_1x02, J3 BARREL_JACK, Q1 IRLB8721PBF, Q2 IRLB8721PBF, Q3 IRLB8721PBF, Q4 IRLB8721PBF, U1 PIC18F45K20-I/PT, U2 IR2110, U3 IR2110, U4 R-78E15, U5 R-78E3.3, U6 XBEE_Wi-Fi

Commit message: Schematics and footprint libraries ready
Parts:
- Cf1, Cr2: value 10nF -> C
- Cf2: value 2.2nF -> C
- Cr1: value 100nF -> C
- D3, D4: value LED -> LED_ALT
Changed lines of the file:
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@@
     (links 127)
     (no_connects 13)
-    (area 57.819999 25.526999 268.528572 193.85)
+    (area 57.819999 25.526999 217.970001 125.725001)
     (thickness 1.6)
     (drawings 53)
@@
       (effects (font (size 1 1) (thickness 0.15)))
     )
-    (fp_text value 10nF (at 7.5 4.31 180) (layer F.Fab)
+    (fp_text value C (at 7.5 4.31 180) (layer F.Fab)
       (effects (font (size 1 1) (thickness 0.15)))
     )
@@
       (effects (font (size 1 1) (thickness 0.15)))
     )
-    (fp_text value 100nF (at 7.5 3.81 180) (layer F.Fab)
+    (fp_text value C (at 7.5 3.81 180) (layer F.Fab)
       (effects (font (size 1 1) (thickness 0.15)))
     )
@@
       (effects (font (size 1 1) (thickness 0.15)))
     )
-    (fp_text value 2.2nF (at 7.5 3.81) (layer F.Fab)
+    (fp_text value C (at 7.5 3.81) (layer F.Fab)
       (effects (font (size 1 1) (thickness 0.15)))
     )
@@
       (effects (font (size 1 1) (thickness 0.15)))
     )
-    (fp_text value 10nF (at 7.5 4.31 180) (layer F.Fab)
+    (fp_text value C (at 7.5 4.31 180) (layer F.Fab)
       (effects (font (size 1 1) (thickness 0.15)))
     )
@@
       (effects (font (size 1 1) (thickness 0.15)))
     )
-    (fp_text value LED (at 1.825 2.95 180) (layer F.Fab)
+    (fp_text value LED_ALT (at 1.825 2.95 180) (layer F.Fab)
       (effects (font (size 1 1) (thickness 0.15)))
     )
@@
       (effects (font (size 1 1) (thickness 0.15)))
     )
-    (fp_text value LED (at -0.025 3 180) (layer F.Fab)
+    (fp_text value LED_ALT (at -0.025 3 180) (layer F.Fab)
       (effects (font (size 1 1) (thickness 0.15)))
     )
@@
   (segment (start 191.948 114.923) (end 193.175 116.15) (width 0.45) (layer F.Cu) (net 70))
   (segment (start 198.475 116.15) (end 198.975 116.65) (width 0.8) (layer F.Cu) (net 70))
-  (segment (start 77.85 34.4) (end 77.85 40.625) (width 4) (layer B.Cu) (net 71))
   (segment (start 77.85 40.625) (end 77.95 40.725) (width 4) (layer B.Cu) (net 71))
   (segment (start 77.95 40.725) (end 77.95 52.675) (width 4) (layer B.Cu) (net 71))
@@
   (segment (start 83.575 72.625) (end 78.05 67.1) (width 4) (layer B.Cu) (net 71))
   (segment (start 70.775 105.5) (end 70.775 41.475) (width 4) (layer B.Cu) (net 71))
-  (segment (start 70.775 41.475) (end 77.85 34.4) (width 4) (layer B.Cu) (net 71))
   (segment (start 74.7 105.375) (end 74.7 37.55) (width 4) (layer B.Cu) (net 71))
-  (segment (start 74.7 37.55) (end 77.85 34.4) (width 4) (layer B.Cu) (net 71))
   (segment (start 63.475 112.25) (end 67.25 112.25) (width 4) (layer B.Cu) (net 71))
   (segment (start 74.125 105.375) (end 74.7 105.375) (width 4) (layer B.Cu) (net 71))
@@
   (segment (start 70.825 112.25) (end 77.85 105.225) (width 4) (layer B.Cu) (net 71))
   (segment (start 77.85 105.225) (end 78 105.375) (width 4) (layer B.Cu) (net 71))
-  (segment (start 77.85 34.4) (end 77.85 105.225) (width 4) (layer B.Cu) (net 71))
   (segment (start 77.85 105.225) (end 78 105.375) (width 4) (layer B.Cu) (net 71))
   (segment (start 85.775 116.35) (end 85.775 72.675) (width 4) (layer B.Cu) (net 71))
@@
   (segment (start 70.775 105.5) (end 70.9 105.375) (width 4) (layer B.Cu) (net 71))
   (segment (start 70.9 105.375) (end 78 105.375) (width 4) (layer B.Cu) (net 71))
+  (segment (start 77.85 34.4) (end 77.85 40.625) (width 4) (layer B.Cu) (net 71))
+  (segment (start 70.775 41.475) (end 77.85 34.4) (width 4) (layer B.Cu) (net 71))
+  (segment (start 74.7 37.55) (end 77.85 34.4) (width 4) (layer B.Cu) (net 71))
+  (segment (start 77.85 34.4) (end 77.85 105.225) (width 4) (layer B.Cu) (net 71))
+  (segment (start 67.85 29.4) (end 62.85 34.4) (width 4) (layer B.Cu) (net 72))
+  (segment (start 84.75 29.4) (end 67.85 29.4) (width 4) (layer B.Cu) (net 72))
+  (segment (start 62.85 34.4) (end 62.85 33.85) (width 4) (layer B.Cu) (net 72))
+  (segment (start 62.85 33.85) (end 67.825 28.875) (width 4) (layer B.Cu) (net 72))
+  (segment (start 67.825 28.875) (end 88.15 28.875) (width 4) (layer B.Cu) (net 72))
+  (segment (start 72.125 29.4) (end 88.675 29.4) (width 4) (layer B.Cu) (net 72))
+  (segment (start 67.825 28.875) (end 88.15 28.875) (width 4) (layer B.Cu) (net 72))
+  (segment (start 65.175 31.525) (end 67.825 28.875) (width 4) (layer B.Cu) (net 72))
+  (segment (start 63 105.375) (end 63 34.55) (width 4) (layer B.Cu) (net 72))
+  (segment (start 63 34.55) (end 62.85 34.4) (width 4) (layer B.Cu) (net 72))
   (segment (start 63 52.725) (end 63 59.775) (width 4) (layer B.Cu) (net 72))
   (segment (start 63 59.775) (end 63.05 59.825) (width 4) (layer B.Cu) (net 72))
@@
   (segment (start 85.725 43.25) (end 87.85 41.125) (width 4) (layer B.Cu) (net 72))
   (segment (start 90.25 34.15) (end 89.5 34.15) (width 4) (layer B.Cu) (net 72))
-  (segment (start 67.85 29.4) (end 62.85 34.4) (width 4) (layer B.Cu) (net 72))
-  (segment (start 84.75 29.4) (end 67.85 29.4) (width 4) (layer B.Cu) (net 72))
   (segment (start 89.5 34.15) (end 84.75 29.4) (width 4) (layer B.Cu) (net 72))
-  (segment (start 62.85 34.4) (end 62.85 33.85) (width 4) (layer B.Cu) (net 72))
-  (segment (start 62.85 33.85) (end 67.825 28.875) (width 4) (layer B.Cu) (net 72))
-  (segment (start 67.825 28.875) (end 88.15 28.875) (width 4) (layer B.Cu) (net 72))
   (segment (start 88.15 28.875) (end 90.25 30.975) (width 4) (layer B.Cu) (net 72))
   (segment (start 85.725 47.875) (end 85.725 45.925) (width 4) (layer B.Cu) (net 72))
@@
   (segment (start 62.95 40.725) (end 62.95 38.575) (width 4) (layer B.Cu) (net 72))
   (segment (start 62.95 38.575) (end 72.125 29.4) (width 4) (layer B.Cu) (net 72))
-  (segment (start 72.125 29.4) (end 88.675 29.4) (width 4) (layer B.Cu) (net 72))
   (segment (start 88.675 29.4) (end 90.25 30.975) (width 4) (layer B.Cu) (net 72))
   (segment (start 63 105.375) (end 63.2 105.375) (width 4) (layer B.Cu) (net 72))
   (segment (start 63.2 105.375) (end 65.175 103.4) (width 4) (layer B.Cu) (net 72))
   (segment (start 88.15 28.875) (end 90.25 30.975) (width 4) (layer B.Cu) (net 72))
-  (segment (start 67.825 28.875) (end 88.15 28.875) (width 4) (layer B.Cu) (net 72))
-  (segment (start 65.175 31.525) (end 67.825 28.875) (width 4) (layer B.Cu) (net 72))
   (segment (start 65.175 103.4) (end 65.175 31.525) (width 4) (layer B.Cu) (net 72))
-  (segment (start 63 105.375) (end 63 34.55) (width 4) (layer B.Cu) (net 72))
-  (segment (start 63 34.55) (end 62.85 34.4) (width 4) (layer B.Cu) (net 72))
   (segment (start 140.6875 62.7625) (end 138.4875 62.7625) (width 0.8) (layer B.Cu) (net 74))
   (segment (start 138.2 63.05) (end 138.2 61.525) (width 0.8) (layer B.Cu) (net 74))
