File: wireless-power-transfer/primary/KiCad/tfg.sch (KiCad schematic (older format))
At the start: 31 parts, among them J1 CONN_01X06, J2 Screw_Terminal_1x02, J3 BARREL_JACK, Q1 IRLB8721PBF, Q2 IRLB8721PBF, Q3 IRLB8721PBF, Q4 IRLB8721PBF, U2 IR2110, U3 IR2110, U4 R-78E15, U5 R-78E3.3, U6 XBEE_Wi-Fi

Commit message: Arranged component-library
Parts:
- removed C1, C2: 0.1uF, symbol C
- removed Cboot1, Cboot2: 0.47uF, symbol C
- removed D3, D4: D, symbol D
- removed U?: PIC18F45K20-I/PT, QFP80P1200X1200X120-44N, symbol PIC18F45K20-I/PT
- added C1, C2: 0.1uF, Capacitors_SMD:C_1206_HandSoldering, symbol C_Small
- added Cboot1, Cboot2: 0.47uF, Capacitors_SMD:C_1206_HandSoldering, symbol C_Small
- added D3, D4: LED, LEDs:LED_D3.0mm, symbol LED-RESCUE-tfg
- added U1: PIC18F45K20-I/PT, componentesGIT:PIC18F45K20, symbol PIC18F45K20-I/PT
- C5, C6, C7: value C -> 10uF; footprint (none) -> Capacitors_SMD:C_1206_HandSoldering
- D1, D2: footprint (none) -> Diodes_THT:D_DO-35_SOD27_P5.08mm_Vertical_AnodeUp
- F1: footprint (none) -> Fuse_Holders_and_Fuses:Fuseholder5x20_horiz_SemiClosed_Casing10x25mm
- J1: footprint (none) -> Pin_Headers:Pin_Header_Angled_1x06_Pitch2.54mm
- J2: footprint (none) -> Connectors_Terminal_Blocks:TerminalBlock_Pheonix_MKDS1.5-2pol
- J3: footprint (none) -> Connectors:BARREL_JACK
- Q1, Q2, Q3, Q4: footprint TO_SOT_Packages_THT:TO-220_Vertical -> componentesGIT:TO-247AC
- R1, R2, Rpu1: footprint (none) -> Resistors_SMD:R_1206_HandSoldering
- SW_MANUAL1, SW_ON_OFF1, SW_POW1: footprint (none) -> componentes:SPDT_Toggle_Switch
- U2, U3: footprint DIL14-1 -> Housings_DIP:DIP-14_W7.62mm; Availability (none) -> Unavailable; Price (none) -> 2.97 USD
- U4, U5: footprint (none) -> componentes:r-78Exx
- U6: footprint (none) -> componentes:XBee_Wi-Fi
Connections:
- wire segments 178 -> 182

Commit message: Schematics and footprint libraries ready
Parts:
- removed D3, D4: LED, LEDs:LED_D3.0mm, symbol LED-RESCUE-tfg
- added D3, D4: LED_ALT, footprint:LED_D3.0mm, symbol LED_ALT
- C1, C2, C5, C6, C7, Cboot1, Cboot2: footprint Capacitors_SMD:C_1206_HandSoldering -> footprint:C_1206_HandSoldering
- D1, D2: footprint Diodes_THT:D_DO-35_SOD27_P5.08mm_Vertical_AnodeUp -> footprint:D_DO-35_SOD27_P5.08mm_Vertical_AnodeUp
- F1: footprint Fuse_Holders_and_Fuses:Fuseholder5x20_horiz_SemiClosed_Casing10x25mm -> footprint:Fuseholder5x20_horiz_SemiClosed_Casing10x25mm
- J1: footprint Pin_Headers:Pin_Header_Angled_1x06_Pitch2.54mm -> footprint:Pin_Header_Angled_1x06_Pitch2.54mm
- J2: footprint Connectors_Terminal_Blocks:TerminalBlock_Pheonix_MKDS1.5-2pol -> footprint:TerminalBlock_Pheonix_MKDS1.5-2pol
- J3: footprint Connectors:BARREL_JACK -> footprint:BARREL_JACK
- Q1, Q2, Q3, Q4: footprint componentesGIT:TO-247AC -> footprint:TO-247AC
- R1, R2, Rpu1: footprint Resistors_SMD:R_1206_HandSoldering -> footprint:R_1206_HandSoldering
- SW_MANUAL1, SW_ON_OFF1, SW_POW1: footprint componentes:SPDT_Toggle_Switch -> footprint:SPDT_Toggle_Switch
- U1: footprint componentesGIT:PIC18F45K20 -> footprint:PIC18F45K20
- U2, U3: footprint Housings_DIP:DIP-14_W7.62mm -> footprint:DIP-14_W7.62mm
- U4, U5: footprint componentes:r-78Exx -> footprint:r-78Exx
- U6: footprint componentes:XBee_Wi-Fi -> footprint:XBee_Wi-Fi
Changed lines of the file:
@@
 EESchema Schematic File Version 2
-LIBS:tfg-rescue
 LIBS:power
 LIBS:device
@@
 LIBS:contrib
 LIBS:valves
-LIBS:IR2110
-LIBS:ITFP260N
-LIBS:PIC18F45K20-I_PT
-LIBS:pickit3
-LIBS:r-78exx
-LIBS:switches
-LIBS:xbee_wi-fi
-LIBS:irlb8721pbf
+LIBS:prymary_lib
 LIBS:tfg-cache
 EELAYER 25 0
@@
 F 0 "U2" H 5250 3050 50  0001 L BNN
 F 1 "IR2110" H 5250 3050 50  0001 L BNN
-F 2 "Housings_DIP:DIP-14_W7.62mm" H 5250 3050 50  0001 L BNN
+F 2 "footprint:DIP-14_W7.62mm" H 5250 3050 50  0001 L BNN
 F 3 "DIP-14 International Rectifier" H 5250 3050 50  0001 L BNN
 F 4 "High and Low Side Driver%2C All High Voltage Pins On One Side%2C Separate Logic and Power Ground%2C Shut-Down" H 5250 3050 50  0001 L BNN "Description"
@@
 F 0 "U3" H 12400 3050 50  0001 L BNN
 F 1 "IR2110" H 12400 3050 50  0001 L BNN
-F 2 "Housings_DIP:DIP-14_W7.62mm" H 12400 3050 50  0001 L BNN
+F 2 "footprint:DIP-14_W7.62mm" H 12400 3050 50  0001 L BNN
 F 3 "DIP-14 International Rectifier" H 12400 3050 50  0001 L BNN
 F 4 "High and Low Side Driver%2C All High Voltage Pins On One Side%2C Separate Logic and Power Ground%2C Shut-Down" H 12400 3050 50  0001 L BNN "Description"
@@
 F 0 "Cboot2" H 11225 2775 50  0000 L CNN
 F 1 "0.47uF" H 11225 2625 50  0000 L CNN
-F 2 "Capacitors_SMD:C_1206_HandSoldering" H 11500 2700 50  0001 C CNN
+F 2 "footprint:C_1206_HandSoldering" H 11500 2700 50  0001 C CNN
 F 3 "" H 11500 2700 50  0001 C CNN
 	1    11500 2700
@@
 F 0 "Cboot1" H 6210 2770 50  0000 L CNN
 F 1 "0.47uF" H 6210 2620 50  0000 L CNN
-F 2 "Capacitors_SMD:C_1206_HandSoldering" H 6200 2700 50  0001 C CNN
+F 2 "footprint:C_1206_HandSoldering" H 6200 2700 50  0001 C CNN
 F 3 "" H 6200 2700 50  0001 C CNN
 	1    6200 2700
@@
 F 0 "D1" H 6550 3250 50  0000 C CNN
 F 1 "D" H 6550 3050 50  0000 C CNN
-F 2 "Diodes_THT:D_DO-35_SOD27_P5.08mm_Vertical_AnodeUp" H 6550 3150 50  0001 C CNN
+F 2 "footprint:D_DO-35_SOD27_P5.08mm_Vertical_AnodeUp" H 6550 3150 50  0001 C CNN
 F 3 "" H 6550 3150 50  0001 C CNN
 	1    6550 3150
@@
 F 0 "D2" H 11150 3250 50  0000 C CNN
 F 1 "D" H 11150 3050 50  0000 C CNN
-F 2 "Diodes_THT:D_DO-35_SOD27_P5.08mm_Vertical_AnodeUp" H 11150 3150 50  0001 C CNN
+F 2 "footprint:D_DO-35_SOD27_P5.08mm_Vertical_AnodeUp" H 11150 3150 50  0001 C CNN
 F 3 "" H 11150 3150 50  0001 C CNN
 	1    11150 3150
@@
 F 0 "U1" H 7764 8009 50  0000 L BNN
 F 1 "PIC18F45K20-I/PT" H 7629 4416 50  0000 L BNN
-F 2 "componentesGIT:PIC18F45K20" H 7950 6350 50  0001 L BNN
+F 2 "footprint:PIC18F45K20" H 7950 6350 50  0001 L BNN
 F 3 "2.16 USD" H 7950 6350 50  0001 L BNN
 F 4 "TQFP-44 10x10x1mm Tray%2C 32KB%2C Flash%2C 1536bytes-RAM%2C 36I/O%2C 8-Bit nanoWatt" H 7950 6350 50  0001 L BNN "Description"
@@
 F 0 "C2" H 3860 6820 50  0000 L CNN
 F 1 "0.1uF" H 3860 6670 50  0000 L CNN
-F 2 "Capacitors_SMD:C_1206_HandSoldering" H 3850 6750 50  0001 C CNN
+F 2 "footprint:C_1206_HandSoldering" H 3850 6750 50  0001 C CNN
 F 3 "" H 3850 6750 50  0001 C CNN
 	1    3850 6750
@@
 F 0 "C1" H 3860 6570 50  0000 L CNN
 F 1 "0.1uF" H 3860 6420 50  0000 L CNN
-F 2 "Capacitors_SMD:C_1206_HandSoldering" H 3850 6500 50  0001 C CNN
+F 2 "footprint:C_1206_HandSoldering" H 3850 6500 50  0001 C CNN
 F 3 "" H 3850 6500 50  0001 C CNN
 	1    3850 6500
@@
 F 0 "J1" H 3850 7800 50  0000 C CNN
 F 1 "CONN_01X06" V 3950 7450 50  0000 C CNN
-F 2 "Pin_Headers:Pin_Header_Angled_1x06_Pitch2.54mm" H 3850 7450 50  0001 C CNN
+F 2 "footprint:Pin_Header_Angled_1x06_Pitch2.54mm" H 3850 7450 50  0001 C CNN
 F 3 "" H 3850 7450 50  0001 C CNN
 	1    3850 7450
@@
 F 0 "U4" H 7650 1200 60  0000 C CNN
 F 1 "R-78E15" H 7850 1600 60  0000 C CNN
-F 2 "componentes:r-78Exx" H 7850 1450 60  0001 C CNN
+F 2 "footprint:r-78Exx" H 7850 1450 60  0001 C CNN
 F 3 "" H 7850 1450 60  0001 C CNN
 	1    7850 1450
@@
 F 0 "U5" H 9900 1250 60  0000 C CNN
 F 1 "R-78E3.3" H 10100 1650 60  0000 C CNN
-F 2 "componentes:r-78Exx" H 10100 1500 60  0001 C CNN
+F 2 "footprint:r-78Exx" H 10100 1500 60  0001 C CNN
 F 3 "" H 10100 1500 60  0001 C CNN
 	1    10100 1500
@@
 F 0 "J3" H 8550 3645 50  0000 C CNN
 F 1 "BARREL_JACK" H 8550 3295 50  0000 C CNN
-F 2 "Connectors:BARREL_JACK" H 8550 3450 50  0001 C CNN
+F 2 "footprint:BARREL_JACK" H 8550 3450 50  0001 C CNN
 F 3 "" H 8550 3450 50  0001 C CNN
 	1    8550 3450
@@
 F 0 "C5" H 7325 1700 50  0000 L CNN
 F 1 "10uF" H 7325 1500 50  0000 L CNN
-F 2 "Capacitors_SMD:C_1206_HandSoldering" H 7338 1450 50  0001 C CNN
+F 2 "footprint:C_1206_HandSoldering" H 7338 1450 50  0001 C CNN
 F 3 "" H 7300 1600 50  0001 C CNN
 	1    7300 1600
@@
 F 0 "C6" H 8275 1800 50  0000 L CNN
 F 1 "10uF" H 8275 1600 50  0000 L CNN
-F 2 "Capacitors_SMD:C_1206_HandSoldering" H 8288 1550 50  0001 C CNN
+F 2 "footprint:C_1206_HandSoldering" H 8288 1550 50  0001 C CNN
 F 3 "" H 8250 1700 50  0001 C CNN
 	1    8250 1700
@@
 F 0 "C7" H 10625 1850 50  0000 L CNN
 F 1 "10uF" H 10625 1650 50  0000 L CNN
-F 2 "Capacitors_SMD:C_1206_HandSoldering" H 10638 1600 50  0001 C CNN
+F 2 "footprint:C_1206_HandSoldering" H 10638 1600 50  0001 C CNN
 F 3 "" H 10600 1750 50  0001 C CNN
 	1    10600 1750
@@
 F 0 "SW_POW1" H 9200 3620 50  0000 C CNN
 F 1 "SW_SPDT" H 9200 3250 50  0000 C CNN
-F 2 "componentes:SPDT_Toggle_Switch" H 9200 3450 50  0001 C CNN
+F 2 "footprint:SPDT_Toggle_Switch" H 9200 3450 50  0001 C CNN
 F 3 "" H 9200 3450 50  0001 C CNN
 	1    9200 3450
@@
 F 0 "F1" V 7730 2550 50  0000 C CNN
 F 1 "Fuse" V 7575 2550 50  0000 C CNN
-F 2 "Fuse_Holders_and_Fuses:Fuseholder5x20_horiz_SemiClosed_Casing10x25mm" V 7580 2550 50  0001 C CNN
+F 2 "footprint:Fuseholder5x20_horiz_SemiClosed_Casing10x25mm" V 7580 2550 50  0001 C CNN
 F 3 "" H 7650 2550 50  0001 C CNN
 	1    7650 2550
@@
 F 0 "SW_MANUAL1" H 5400 6920 50  0000 C CNN
 F 1 "SW_SPDT" H 5400 6550 50  0000 C CNN
-F 2 "componentes:SPDT_Toggle_Switch" H 5400 6750 50  0001 C CNN
+F 2 "footprint:SPDT_Toggle_Switch" H 5400 6750 50  0001 C CNN
 F 3 "" H 5400 6750 50  0001 C CNN
 	1    5400 6750
@@
 F 0 "SW_ON_OFF1" H 5400 7370 50  0000 C CNN
 F 1 "SW_SPDT" H 5400 7000 50  0000 C CNN
-F 2 "componentes:SPDT_Toggle_Switch" H 5400 7200 50  0001 C CNN
+F 2 "footprint:SPDT_Toggle_Switch" H 5400 7200 50  0001 C CNN
 F 3 "" H 5400 7200 50  0001 C CNN
 	1    5400 7200
@@
 F 0 "U6" H 12900 5850 60  0000 C CNN
 F 1 "XBEE_Wi-Fi" V 11600 5850 60  0000 C CNN
-F 2 "componentes:XBee_Wi-Fi" H 12100 5850 60  0001 C CNN
+F 2 "footprint:XBee_Wi-Fi" H 12100 5850 60  0001 C CNN
 F 3 "" H 12100 5850 60  0001 C CNN
 	1    12100 5850
@@
 NoConn ~ 11850 5350
 $Comp
-L LED-RESCUE-tfg D3
-U 1 1 59E8E0C4
-P 10650 5200
-F 0 "D3" H 10650 5300 50  0000 C CNN
-F 1 "LED" H 10650 5100 50  0000 C CNN
-F 2 "LEDs:LED_D3.0mm" H 10650 5200 50  0001 C CNN
-F 3 "" H 10650 5200 50  0001 C CNN
-	1    10650 5200
-	-1   0    0    1
-$EndComp
-$Comp
-L LED-RESCUE-tfg D4
-U 1 1 59E8E153
-P 10650 5500
-F 0 "D4" H 10650 5600 50  0000 C CNN
-F 1 "LED" H 10650 5400 50  0000 C CNN
-F 2 "LEDs:LED_D3.0mm" H 10650 5500 50  0001 C CNN
-F 3 "" H 10650 5500 50  0001 C CNN
-	1    10650 5500
-	-1   0    0    1
-$EndComp
-$Comp
 L R R1
 U 1 1 59E8E857
@@
 F 0 "R1" V 10330 5200 50  0000 C CNN
 F 1 "R" V 10250 5200 50  0000 C CNN
-F 2 "Resistors_SMD:R_1206_HandSoldering" V 10180 5200 50  0001 C CNN
+F 2 "footprint:R_1206_HandSoldering" V 10180 5200 50  0001 C CNN
 F 3 "" H 10250 5200 50  0001 C CNN
 	1    10250 5200
@@
 F 0 "R2" V 10330 5500 50  0000 C CNN
 F 1 "R" V 10250 5500 50  0000 C CNN
-F 2 "Resistors_SMD:R_1206_HandSoldering" V 10180 5500 50  0001 C CNN
+F 2 "footprint:R_1206_HandSoldering" V 10180 5500 50  0001 C CNN
 F 3 "" H 10250 5500 50  0001 C CNN
 	1    10250 5500
@@
 F 0 "Q1" H 7550 2375 50  0000 L CNN
 F 1 "IRLB8721PBF" H 7550 2300 50  0000 L CNN
-F 2 "componentesGIT:TO-247AC" H 7550 2225 50  0001 L CIN
+F 2 "footprint:TO-247AC" H 7550 2225 50  0001 L CIN
 F 3 "" H 7300 2300 50  0001 L CNN
 	1    7300 2300
@@
 F 0 "Q2" H 7550 3575 50  0000 L CNN
 F 1 "IRLB8721PBF" H 7550 3500 50  0000 L CNN
-F 2 "componentesGIT:TO-247AC" H 7550 3425 50  0001 L CIN
+F 2 "footprint:TO-247AC" H 7550 3425 50  0001 L CIN
 F 3 "" H 7300 3500 50  0001 L CNN
 	1    7300 3500
@@
 F 0 "Q3" H 10650 2375 50  0000 L CNN
 F 1 "IRLB8721PBF" H 10650 2300 50  0000 L CNN
-F 2 "componentesGIT:TO-247AC" H 10650 2225 50  0001 L CIN
+F 2 "footprint:TO-247AC" H 10650 2225 50  0001 L CIN
 F 3 "" H 10400 2300 50  0001 L CNN
 	1    10400 2300
@@
 F 0 "Q4" H 10650 3575 50  0000 L CNN
 F 1 "IRLB8721PBF" H 10650 3500 50  0000 L CNN
-F 2 "componentesGIT:TO-247AC" H 10650 3425 50  0001 L CIN
+F 2 "footprint:TO-247AC" H 10650 3425 50  0001 L CIN
 F 3 "" H 10400 3500 50  0001 L CNN
 	1    10400 3500
@@
 F 0 "J2" H 9200 2400 50  0000 C TNN
 F 1 "Screw_Terminal_1x02" V 9050 2150 50  0000 C TNN
-F 2 "Connectors_Terminal_Blocks:TerminalBlock_Pheonix_MKDS1.5-2pol" H 9200 1925 50  0001 C CNN
+F 2 "footprint:TerminalBlock_Pheonix_MKDS1.5-2pol" H 9200 1925 50  0001 C CNN
 F 3 "" H 9175 2150 50  0001 C CNN
 	1    9200 2150
@@
 F 0 "Rpu1" V 4380 7125 50  0000 C CNN
 F 1 "10k" V 4300 7125 50  0000 C CNN
-F 2 "Resistors_SMD:R_1206_HandSoldering" V 4230 7125 50  0001 C CNN
+F 2 "footprint:R_1206_HandSoldering" V 4230 7125 50  0001 C CNN
 F 3 "" H 4300 7125 50  0001 C CNN
 	1    4300 7125
@@
 	9400 2700 9400 2500
 Connection ~ 9400 2500
+$Comp
+L LED_ALT D3
+U 1 1 5AA74DF4
+P 10650 5200
+F 0 "D3" H 10650 5300 50  0000 C CNN
+F 1 "LED_ALT" H 10650 5100 50  0000 C CNN
+F 2 "footprint:LED_D3.0mm" H 10650 5200 50  0001 C CNN
+F 3 "" H 10650 5200 50  0001 C CNN
+	1    10650 5200
+	-1   0    0    1
+$EndComp
+$Comp
+L LED_ALT D4
+U 1 1 5AA74EA1
+P 10650 5500
+F 0 "D4" H 10650 5600 50  0000 C CNN
+F 1 "LED_ALT" H 10650 5400 50  0000 C CNN
+F 2 "footprint:LED_D3.0mm" H 10650 5500 50  0001 C CNN
+F 3 "" H 10650 5500 50  0001 C CNN
+	1    10650 5500
+	-1   0    0    1
+$EndComp
 $EndSCHEMATC
