File: wireless-power-transfer/secondary/KiCad/secondary.kicad_pcb (KiCad board)
At the start: 2 copper layers, 100 x 57.8 mm, 10 parts, among them J1 Screw_Terminal_1x02, J2 Screw_Terminal_1x02, U1 LM7812CT

Commit message: Secondary libraries arranged
Parts:
- moved Cr1 36.9 mm to (105.8, 124.5)
- moved D1 36.9 mm to (94.0, 97.0)
- moved D2 36.9 mm to (114.0, 97.0)
- moved D3 36.9 mm to (94.0, 89.0)
- moved D4 36.9 mm to (114.0, 89.0)
- moved G*** 36.9 mm to (110.5, 106.7)
- moved J2 36.9 mm to (121.0, 134.0)
- moved U1 36.9 mm to (121.0, 125.0)
- moved Cf1 36.9 mm to (112.5, 132.7)
- moved J1 36.9 mm to (98.8, 133.4)
Other:
- board text added: "6/7"
- board text removed: "DTE"
